File: USB_TOOL.kicad_pcb (KiCad board)
At the start: 2 copper layers, 37 parts, among them J1 USB_Mini_B, J2 PA Connector, J3 PA Connector, J4 PA Connector, U1 ESP32-C3-WROOM-02-N4, U2 3.3V Regurator, U3 5V isolated DC/DC, U4 USB isolatar, U5 FIN1019MTCX

Commit message: 56789
Parts:
- added D1: Green LED, LED_SMD:LED_0603_1608Metric, F.Cu at (93.4, 52.1)
- added D2: Amber LED, LED_SMD:LED_0603_1608Metric, F.Cu at (114.8, 54.1)
- added D3: Orange LED, LED_SMD:LED_0603_1608Metric, F.Cu at (118.9, 54.1)
- added R10: 1k, Resistor_SMD:R_0603_1608Metric, F.Cu at (93.4, 55.1)
- added R11: 1k, Resistor_SMD:R_0603_1608Metric, F.Cu at (114.8, 57.2)
- added R12: 1k, Resistor_SMD:R_0603_1608Metric, F.Cu at (119.0, 57.1)
- C13, C14: moved to B.Cu
- moved C11 64.3 mm to (147.9, 93.2), turned to 90 degrees
- moved C12 63.1 mm to (145.8, 94.4), turned to 90 degrees
- moved R8 60.7 mm to (141.3, 94.4), turned to -90 degrees
- moved J2 60.0 mm to (141.5, 56.3)
- moved U1 54.7 mm to (130.8, 91.0), turned to 180 degrees
- moved C15 53.3 mm to (144.9, 91.8), turned to 180 degrees
- moved R5 37.9 mm to (154.1, 93.9), turned to 90 degrees
- moved SW2 35.7 mm to (163.6, 93.2), turned to 90 degrees
- moved C14 34.3 mm to (163.6, 90.0), turned to 90 degrees
- moved U5 33.2 mm to (171.7, 68.8), turned to 90 degrees
- moved SW1 29.3 mm to (157.0, 93.2), turned to 90 degrees
- moved J4 29.2 mm to (155.6, 56.3)
- moved R9 28.5 mm to (172.7, 64.3), turned to 0 degrees
- moved C16 27.5 mm to (166.5, 68.3), turned to -90 degrees
- moved J3 26.7 mm to (171.6, 56.3)
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Routing:
- net GND1: track 0.00 -> 35.0 mm, vias 0 -> 1
- net EN: track 0.00 -> 29.3 mm, vias 0 -> 1
- net VBUS: track 0.00 -> 27.8 mm
- net BOOT: track 0.00 -> 25.9 mm, vias 0 -> 2
- net GND2: track 0.00 -> 20.3 mm
- net Net-(U4-PIN): track 0.00 -> 12.8 mm
- net Net-(U4-PDEN): track 0.00 -> 11.9 mm
- net +3.3V: track 0.00 -> 8.62 mm
- net UD-: track 0.00 -> 7.34 mm
- net Net-(U3-Vin+): track 0.00 -> 6.88 mm
- net +5V: track 0.00 -> 6.75 mm
- net UD+: track 0.00 -> 6.63 mm
- net Net-(U4-UD-): track 0.00 -> 3.05 mm
- net Net-(U4-UD+): track 0.00 -> 3.05 mm
Other:
- board outline added: 100 x 45.9 mm
- board text added: "BOOT"
- board text added: "EN"
- board text added: "I2C"
- board text added: "LVDS"
- board text added: "SPI"

Commit message: ASD
Parts:
- added C17: 0.1uF, Capacitor_SMD:C_0603_1608Metric, F.Cu at (148.0, 71.3)
- added C18: 0.1uF, Capacitor_SMD:C_0603_1608Metric, F.Cu at (152.1, 64.5)
- added G***: LOGO, global_footprints:icon_small_16.0x10.0, F.Cu at (85.6, 89.3)
- added J5: PA Connector, S02B-PASK-2:S02B-PASK-2, F.Cu at (129.5, 56.3)
- added J6: Conn_01x02_Socket, Connector_PinHeader_2.54mm:PinHeader_1x02_P2.54mm_Vertical, F.Cu at (130.8, 64.1)
- added J7: PA Connector, S02B-PASK-2:S02B-PASK-2, F.Cu at (148.0, 56.3)
- added R13: 100, Resistor_SMD:R_0402_1005Metric, B.Cu at (148.0, 66.8)
- added R14: 100, Resistor_SMD:R_0402_1005Metric, B.Cu at (148.0, 65.8)
- added R15: 10k, Resistor_SMD:R_0603_1608Metric, F.Cu at (143.8, 63.7)
- added R16: 10k, Resistor_SMD:R_0603_1608Metric, F.Cu at (117.7, 56.4)
- added U6: CAN transceiver, Package_SO:SOIC-8_3.9x4.9mm_P1.27mm, F.Cu at (148.0, 66.2)
- J2: footprint S02B-PASK-2:S02B-PASK-2 -> S04B-PASK-2:S04B-PASK-2
- J4: footprint S04B-PASK-2:S04B-PASK-2 -> S02B-PASK-2:S02B-PASK-2
- moved J2 30.1 mm to (171.6, 56.3)
- moved R4 24.8 mm to (119.8, 89.2)
- moved R3 24.5 mm to (119.8, 87.7)
- moved R6 23.7 mm to (143.1, 86.2), turned to 180 degrees
- moved R7 19.0 mm to (114.7, 93.1)
- moved J4 17.6 mm to (138.0, 56.3)
- moved J3 12.6 mm to (159.1, 56.3)
- moved D2 12.0 mm to (103.0, 52.1)
- moved R11 11.9 mm to (103.0, 55.1)
- moved C7 10.7 mm to (120.7, 53.6)
- moved R12 10.0 mm to (109.1, 55.1)
- moved D3 10.00 mm to (109.1, 52.1)
- moved U2 9.87 mm to (117.3, 53.6)
- moved C6 9.85 mm to (113.8, 53.6)
- moved C16 2.24 mm to (168.1, 66.7)
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Connections:
- net Net-(U4-DD+) renamed /U4_DD+
- net Net-(U4-DD-) renamed /U4_DD-
- J2 pad 1: I2C_SCL -> LVDS_DO+
- J2 pad 2: I2C_SDA -> LVDS_DO-
- J3 pad 1: LVDS_RI- -> SPI_SS
- J3 pad 2: LVDS_RI+ -> SPI_SDO
- J3 pad 3: LVDS_DO- -> SPI_SDI
- J3 pad 4: LVDS_DO+ -> SPI_SCK
- J4 pad 1: SPI_SCK -> I2C_SCL
- J4 pad 2: SPI_SDI -> I2C_SDA
- U1 pad 19: unconnected-(U1-GND-Pad19) -> GND2
- U2 pad 3: unconnected-(U2-EN-Pad3) -> Net-(U2-EN)
- U5 pad 7: unconnected-(U5-GND-Pad7) -> GND2
Routing:
- net GND2: track 20.3 -> 272.5 mm, vias 0 -> 355
- net +3.3V: track 8.62 -> 208.0 mm, vias 0 -> 15
- net +5V: track 6.75 -> 104.4 mm, vias 0 -> 4
- net SPI_SCK: track 0.00 -> 89.3 mm, vias 0 -> 2
- net SPI_SDO: track 0.00 -> 76.6 mm, vias 0 -> 2
- net LVDS_RE: track 0.00 -> 75.3 mm
- net LVDS_DE: track 0.00 -> 74.8 mm, vias 0 -> 2
- net LVDS_DI: track 0.00 -> 68.6 mm
- net LVDS_RO: track 0.00 -> 67.0 mm
- net I2C_SCL: track 0.00 -> 53.6 mm, vias 0 -> 3
- net SPI_SS: track 0.00 -> 43.8 mm, vias 0 -> 1
- net SPI_SDI: track 0.00 -> 43.5 mm, vias 0 -> 1
- net /U4_DD+: track 0.00 -> 34.6 mm
- net /U4_DD-: track 0.00 -> 34.2 mm
- net I2C_SDA: track 0.00 -> 32.6 mm, vias 0 -> 1
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- added copper zone on B.Cu, net GND1
- added copper zone on F.Cu, net GND1
- added copper zone on B.Cu, net GND2
- added copper zone on F.Cu, net GND2
Other:
- board text added: "CAN"
- board text added: "POWER"
- board text added: "USB TOOL"

Commit message: update
Connections:
- net Net-(U6-CANH) renamed CAN+
- net Net-(U6-CANL) renamed CAN-
Routing:
- net GND2: track 272.5 -> 289.4 mm, vias 355 -> 345
- net (no net): vias 2 -> 0

Commit message: update
Parts:
- added REF**: MountingHole_3.2mm_M3_DIN965, MountingHole:MountingHole_3.2mm_M3_DIN965, F.Cu at (81.8, 54.2)
- added REF**: MountingHole_3.2mm_M3_DIN965, MountingHole:MountingHole_3.2mm_M3_DIN965, F.Cu at (81.8, 81.2)
- added REF**: MountingHole_3.2mm_M3_DIN965, MountingHole:MountingHole_3.2mm_M3_DIN965, F.Cu at (171.8, 91.2)
